Commit message: add rxbot pose env

File: pybullet_wrapper/assets/r5.urdf (robot description, URDF)
Before this commit: robot r2, 7 links, 6 joints
Joints:
- joint ee: origin xyz=0 0 0.15 rpy=0 -1.570795 3.141592 -> xyz=0 0 0.1 rpy=0 -1.570795 3.141592

File: pybullet_wrapper/assets/r6.urdf (robot description, URDF)
Before this commit: robot r2, 6 links, 5 joints
Links:
- added link link5, mass 1; collision box size=0.05 0.05 0.1; visual box size=0.05 0.05 0.1
- added link link6, mass 1; collision box size=0.05 0.05 0.1; visual box size=0.05 0.05 0.1
Joints:
- added joint joint5: type revolute, parent link4, child link5, origin xyz=0 0 0.1 rpy=0 0 0, axis 0 0 1, limit lower=-2.36 upper=2.36 effort=30 velocity=1.0
- added joint joint6: type revolute, parent link5, child link6, origin xyz=0 0 0.1 rpy=0 0 0, axis 1 0 0, limit lower=-2.36 upper=2.36 effort=30 velocity=1.0
- joint ee: parent link4 -> link6

File: pybullet_wrapper/assets/r7.urdf (robot description, URDF)
Before this commit: robot r2, 6 links, 5 joints
Links:
- added link link5, mass 1; collision box size=0.05 0.05 0.1; visual box size=0.05 0.05 0.1
- added link link6, mass 1; collision box size=0.05 0.05 0.1; visual box size=0.05 0.05 0.1
- added link link7, mass 1; collision box size=0.05 0.05 0.1; visual box size=0.05 0.05 0.1
Joints:
- added joint joint5: type revolute, parent link4, child link5, origin xyz=0 0 0.1 rpy=0 0 0, axis 0 0 1, limit lower=-2.36 upper=2.36 effort=30 velocity=1.0
- added joint joint6: type revolute, parent link5, child link6, origin xyz=0 0 0.1 rpy=0 0 0, axis 1 0 0, limit lower=-2.36 upper=2.36 effort=30 velocity=1.0
- added joint joint7: type revolute, parent link6, child link7, origin xyz=0 0 0.1 rpy=0 0 0, axis 0 0 1, limit lower=-2.36 upper=2.36 effort=30 velocity=1.0
- joint ee: parent link4 -> link7
